File: nrom-128/nrom-128.kicad_sch (KiCad schematic)
At the start: 5 parts, among them J1 NES_Cart_Edge, U1 27C512, U2 27C512, U3 ATtiny13A-PU

Commit message: protoboard rev 0
Parts:
- C1: footprint SamacSys_Parts:104MSR400K -> Library:film-cap
Changed lines of the file:
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@@
       (effects (font (size 1.27 1.27)) (justify left))
     )
-    (property "Footprint" "SamacSys_Parts:104MSR400K" (id 2) (at 236.22 120.65 0)
+    (property "Footprint" "Library:film-cap" (id 2) (at 236.22 120.65 0)
       (effects (font (size 1.27 1.27)) (justify left) hide)
     )
@@
     )
     (path "/e89ce05c-67ba-427f-8e6b-c188ac5f7391"
-      (reference "C1") (unit 1) (value "100nF") (footprint "SamacSys_Parts:104MSR400K")
+      (reference "C1") (unit 1) (value "100nF") (footprint "Library:film-cap")
     )
     (path "/00000000-0000-0000-0000-0000632ebbec"
