File: nrom-128/nrom-128.kicad_pcb (KiCad board)
At the start: 2 copper layers, 99 x 40 mm, 5 parts, among them J1 NES_Cart_Edge, U1 8kb CHR, U2 16kb PRG, U3 Anti-Lock

Commit message: PCB edge connector corrected
Parts:
- added G***: LOGO, Library:nrom-badge, F.Cu at (162.0, 96.0)
Routing:
- net /CHR_A10: track 41.0 -> 40.2 mm
- net /PRG_A11: track 27.8 -> 28.5 mm
- net VCC: track 144.5 -> 145.0 mm
- net /PRG_OE: vias 3 -> 2

Commit message: protoboard rev 0
Parts:
- added G***: LOGO, Library:back-screen-protoboard, B.Cu at (159.0, 87.0)
- C1: value Film Cap -> 100nF; footprint SamacSys_Parts:104MSR400K -> Library:film-cap
- moved C1 5.39 mm to (120.5, 78.0)
- moved G*** 2.50 mm to (159.5, 96.0)
Other:
- board text added: "100nF Film Cap"

Commit message: pcb mods
Parts:
- removed the G*** at (159.0, 87.0)
- added G***: LOGO, Library:back-screen-hand-soldered, B.Cu at (159.0, 87.0)

Commit message: manually soldered PCB
Parts:
- removed the G*** at (159.0, 87.0)
- added G***: LOGO, Library:back-screen-manually-soldered, B.Cu at (159.0, 87.0)
- added kibuzzard-63F70D0C: G***, kibuzzard-63F70D0C, F.Cu at (205.5, 84.0)
- added kibuzzard-63F70D54: G***, kibuzzard-63F70D54, F.Cu at (117.0, 96.0)
- added kibuzzard-63F70D89: G***, kibuzzard-63F70D89, F.Cu at (121.0, 77.0)
- added kibuzzard-63F7105E: G***, kibuzzard-63F7105E, F.Cu at (129.0, 84.0)
- added kibuzzard-63F711A0: G***, kibuzzard-63F711A0, F.Cu at (121.0, 79.5)
Other:
- board text removed: "100nF Film Cap"
